Commit message: Updated puma560_description.urdf file

File: urdf/puma560_description.urdf (robot description, URDF)
Before this commit: robot puma560_description, 6 links, 5 joints
Links:
- link base_link: geometry collision mesh filename=package://puma560_description/meshes/puma560_base_link.STL; visual mesh filename=package://puma560_description/meshes/puma560_base_link.STL
- link elbow_link: geometry collision mesh filename=package://puma560_description/meshes/puma560_elbow_link.STL; visual mesh filename=package://puma560_description/meshes/puma560_elbow_link.STL
- link shoulder_link: geometry collision mesh filename=package://puma560_description/meshes/puma560_shoulder_link.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; visual mesh filename=package://puma560_description/meshes/puma560_shoulder_link.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
- link waist_link: geometry collision mesh filename=package://puma560_description/meshes/puma560_waist_link.STL; visual mesh filename=package://puma560_description/meshes/puma560_waist_link.STL
- link wrist_bend_link: geometry collision mesh filename=package://puma560_description/meshes/puma560_wrist_bend_lin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; visual mesh filename=package://puma560_description/meshes/puma560_wrist_bend_lin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
- link wrist_roll_link: geometry collision mesh filename=package://puma560_description/meshes/puma560_wrist_roll_lin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; visual mesh filename=package://puma560_description/meshes/puma560_wrist_roll_lin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
