Commit message: Updated urdf file with elbow link CS orientation

File: urdf/puma560_description.old.urdf (robot description, URDF)
Before this commit: robot puma560_description, 6 links, 5 joints
Joints:
- joint elbow_wrist_roll_joint: origin xyz=0.43209 0 0 rpy=0.011076 0 0 -> xyz=0.43209 0 0 rpy=-3.1305 0 0
- joint shoulder_elbow_link: axis 0 1 0 -> 0 -1 0; origin xyz=0.4318 0.0889 0 rpy=0 0.02129 0 -> xyz=0.4318 0.0889 0 rpy=3.1416 0.057886 0
- joint waist_shoulder_joint: origin xyz=0 -0.21844 0 rpy=0 -0.046426 0 -> xyz=0 -0.21844 0 rpy=0 -0.083022 0
- joint wrist_roll_bend_joint: origin xyz=0 0 0 rpy=0 -0.14699 0 -> xyz=0 0 0 rpy=0 -0.19722 0
